File: Documentation/Schematic/ALF.sch (KiCad schematic (older format))
At the start: 0 parts

Commit message: Updated schematic
Parts:
- added D? (x4): LED, symbol LED
- added JP1, JP7: CONN_02X20, symbol CONN_02X20
- added JP2: CONN_02X03, symbol CONN_02X03
- added JP3, JP6: CONN_01X08, symbol CONN_01X08
- added JP4: CONN_01X10, symbol CONN_01X10
- added JP5: CONN_01X06, symbol CONN_01X06
- added P?: CONN_02X05, symbol CONN_02X05
- added P?: CONN_02X07, symbol CONN_02X07
- added P? (x4): CONN_01X05, symbol CONN_01X05
- added P?: CONN_01X24, symbol CONN_01X24
- added R? (x4): R, symbol R
Connections:
- new net: D?.2 (A), R?.1 (x4)
- new net AD0: P?.9 (P9)
- new net ADC_IN0: JP5.1 (P1)
- new net ADC_IN1: JP5.2 (P2)
- new net ADC_IN2: JP5.3 (P3)
- new net ADC_IN3: JP5.4 (P4)
- new net ADC_IN4: JP5.5 (P5)
- new net ADC_IN5: JP5.6 (P6)
- new net AUX_CL: P?.7 (P7)
- new net AUX_DA: P?.6 (P6)
- new net Arduino_IO0: JP3.8 (P8), JP6.8 (P8)
- new net Arduino_IO1: JP3.7 (P7), JP6.7 (P7)
- new net Arduino_IO10: JP4.8 (P8)
- new net Arduino_IO11: JP2.4 (P4), JP4.7 (P7)
- new net Arduino_IO12: JP2.1 (P1), JP4.6 (P6)
- new net Arduino_IO13: JP2.3 (P3), JP4.5 (P5)
- new net Arduino_IO14: JP4.2 (P2)
- new net Arduino_IO15: JP4.1 (P1)
- new net Arduino_IO2: JP3.6 (P6), JP6.6 (P6)
- new net Arduino_IO3: JP3.5 (P5), JP6.5 (P5)
- new net Arduino_IO4: JP3.4 (P4), JP6.4 (P4)
- new net Arduino_IO5: JP3.3 (P3), JP6.3 (P3)
- new net Arduino_IO6: JP3.2 (P2), JP6.2 (P2)
- new net Arduino_IO7: JP3.1 (P1), JP6.1 (P1)
- new net Arduino_IO8: JP4.10 (P10)
- new net Arduino_IO9: JP4.9 (P9)
- new net Arduino_Reset_n: JP2.5 (P5)
- new net Arduino_VREF: JP4.3 (P3)
- new net CLKIN: P?.1 (P1)
- new net CPOUT: P?.20 (P20)
- new net FSYNC: P?.11 (P11)
- new net GND: D?.1 (K), D?.1 (K), D?.1 (K), D?.1 (K), JP1.12 (P12), JP1.30 (P30), JP2.6 (P6), JP4.4 (P4), JP7.12 (P12), JP7.30 (P30), P?.18 (P18), P?.5 (P5), P?.5 (P5), P?.5 (P5), P?.5 (P5)
- new net GPIO_0_D0: JP1.1 (P1)
- new net GPIO_0_D1: JP1.2 (P2)
- new net GPIO_0_D10: JP1.13 (P13)
- new net GPIO_0_D11: JP1.14 (P14)
- new net GPIO_0_D12: JP1.15 (P15)
- new net GPIO_0_D13: JP1.16 (P16)
- new net GPIO_0_D14: JP1.17 (P17)
- new net GPIO_0_D15: JP1.18 (P18)
- new net GPIO_0_D16: JP1.19 (P19)
- new net GPIO_0_D17: JP1.20 (P20)
- new net GPIO_0_D18: JP1.21 (P21)
- new net GPIO_0_D19: JP1.22 (P22)
- new net GPIO_0_D2: JP1.3 (P3)
- new net GPIO_0_D20: JP1.23 (P23)
- new net GPIO_0_D21: JP1.24 (P24)
- new net GPIO_0_D22: JP1.25 (P25)
- new net GPIO_0_D23: JP1.26 (P26)
- new net GPIO_0_D24: JP1.27 (P27)
- new net GPIO_0_D25: JP1.28 (P28)
- new net GPIO_0_D26: JP1.31 (P31)
- new net GPIO_0_D27: JP1.32 (P32)
- new net GPIO_0_D28: JP1.33 (P33)
- new net GPIO_0_D29: JP1.34 (P34)
- new net GPIO_0_D3: JP1.4 (P4)
- new net GPIO_0_D30: JP1.35 (P35)
- new net GPIO_0_D31: JP1.36 (P36)
- new net GPIO_0_D32: JP1.37 (P37)
- new net GPIO_0_D33: JP1.38 (P38)
- new net GPIO_0_D34: JP1.39 (P39)
- new net GPIO_0_D35: JP1.40 (P40)
- new net GPIO_0_D4: JP1.5 (P5)
- new net GPIO_0_D5: JP1.6 (P6)
- new net GPIO_0_D6: JP1.7 (P7)
- new net GPIO_0_D7: JP1.8 (P8)
- new net GPIO_0_D8: JP1.9 (P9)
- new net GPIO_0_D9: JP1.10 (P10)
- new net GPIO_1_D0: JP7.1 (P1)
- new net GPIO_1_D1: JP7.2 (P2)
- new net GPIO_1_D10: JP7.13 (P13)
- new net GPIO_1_D11: JP7.14 (P14)
- new net GPIO_1_D12: JP7.15 (P15)
- new net GPIO_1_D13: JP7.16 (P16)
- new net GPIO_1_D14: JP7.17 (P17)
- new net GPIO_1_D15: JP7.18 (P18)
- new net GPIO_1_D16: JP7.19 (P19)
- new net GPIO_1_D17: JP7.20 (P20)
- new net GPIO_1_D18: JP7.21 (P21)
- new net GPIO_1_D19: JP7.22 (P22)
- new net GPIO_1_D2: JP7.3 (P3)
- new net GPIO_1_D20: JP7.23 (P23)
- new net GPIO_1_D21: JP7.24 (P24)
- new net GPIO_1_D22: JP7.25 (P25)
- new net GPIO_1_D23: JP7.26 (P26)
- new net GPIO_1_D24: JP7.27 (P27)
- new net GPIO_1_D25: JP7.28 (P28)
- new net GPIO_1_D26: JP7.31 (P31)
- new net GPIO_1_D27: JP7.32 (P32)
- new net GPIO_1_D28: JP7.33 (P33)
- new net GPIO_1_D29: JP7.34 (P34)
- new net GPIO_1_D3: JP7.4 (P4)
- new net GPIO_1_D30: JP7.35 (P35)
- new net GPIO_1_D31: JP7.36 (P36)
- new net GPIO_1_D32: JP7.37 (P37)
- new net GPIO_1_D33: JP7.38 (P38)
- new net GPIO_1_D34: JP7.39 (P39)
- new net GPIO_1_D35: JP7.40 (P40)
- new net GPIO_1_D4: JP7.5 (P5)
- new net GPIO_1_D5: JP7.6 (P6)
- new net GPIO_1_D6: JP7.7 (P7)
- new net GPIO_1_D7: JP7.8 (P8)
- new net GPIO_1_D8: JP7.9 (P9)
- new net GPIO_1_D9: JP7.10 (P10)
- new net INT: P?.12 (P12)
- new net REGOUT: P?.10 (P10)
- new net RESV: P?.19 (P19), P?.21 (P21), P?.22 (P22)
- new net SCL: P?.23 (P23)
- new net SCL_U1: P?.3 (P3)
- new net SCL_U2: P?.3 (P3)
- new net SCL_U3: P?.3 (P3)
- new net SCL_U4: P?.3 (P3)
- new net SDA: P?.24 (P24)
- new net SDA_U1: P?.2 (P2)
- new net SDA_U2: P?.2 (P2)
- new net SDA_U3: P?.2 (P2)
- new net SDA_U4: P?.2 (P2)
- new net VCC: P?.1 (P1), P?.1 (P1), P?.1 (P1), P?.1 (P1)
- new net VCC3P3: JP1.29 (P29), JP7.29 (P29)
- new net VCC5: JP1.11 (P11), JP2.2 (P2), JP7.11 (P11)
- new net VDD: P?.13 (P13)
- new net VLOGIC: P?.8 (P8)
Other:
- note added: "Beleuchtung"
- note added: "Buttons"
- note added: "Display"
- note added: "Drehzahlsensor"
- note added: "Levelshifter"
- note added: "MPU 6050"
- note added: "Motortreiber"
- note added: "Ultraschall SRF08"

Commit message: Updated Schematics
Parts:
- removed D? (x4): LED, symbol LED
- removed P? (x4): CONN_01X05, symbol CONN_01X05
- removed P?: CONN_01X24, symbol CONN_01X24
- removed R? (x4): R, symbol R
- added CON?: BARREL_JACK, symbol BARREL_JACK
- added P?: CONN_AKKU, symbol CONN_01X02
- added P?: CONN_01X08, symbol CONN_01X08
- added P?: CONN_01X04, symbol CONN_01X04
- added R?: 120, symbol R
Connections:
- net labels added: ADC_IN6, ADC_IN7, AKKU+, LED_HL_IN, LED_HL_OUT, LED_HR_IN, LED_HR_OUT, LED_VL_IN, LED_VL_OUT, LED_VR_IN, LED_VR_OUT, MISO, MISO_5V, MOSI, MOSI_5V, MOTOR_A, MOTOR_B, MOTOR_DIR_33, MOTOR_DIR_5V, MOTOR_PWM_33, MOTOR_PWM_5V, MPU6050_AD0, MPU6050_INT, MPU6050_XCL, MPU6050_XDA, ROT_OUT, SCLK, SCLK_5V, SCL_5V, SDA_5V, SD_CS, SD_CS_5V, TFT_CS, TFT_CS_5V, TFT_DC, TFT_DC_5V, TOUCH_CS, TOUCH_CS_5V, VCC33, VCC9, VCC_33, VCC_5
- net labels removed: AD0, AUX_CL, AUX_DA, Arduino_IO10, Arduino_IO4, Arduino_IO8, Arduino_IO9, CLKIN, CPOUT, FSYNC, GPIO_1_D0, GPIO_1_D1, GPIO_1_D2, GPIO_1_D3, GPIO_1_D4, GPIO_1_D5, GPIO_1_D6, GPIO_1_D7, INT, REGOUT, RESV, SCL_U1, SCL_U2, SCL_U3, SCL_U4, SDA_U1, SDA_U2, SDA_U3, SDA_U4, VCC, VDD, VLOGIC
- wire segments 1 -> 82
Other:
- note added: "Spannungsversorgung FPGA"
- note added: "Spannungswandler"
- note removed: "Buttons"
- moved on the sheet: JP7, P?

Commit message: Updated Schematic (Removed levelshifter on SPI Pins and added I2C pullup)
Connections:
- net labels removed: MISO_5V, MOSI_5V, SCLK_5V, SD_CS_5V, TFT_CS_5V, TFT_DC_5V, TOUCH_CS_5V
- wire segments 82 -> 73
Changed lines of the file:
@@
 VCC_5
 Wire Wire Line
-	8100 4300 8100 4400
+	8100 4300 8100 4350
+Wire Wire Line
+	8100 4350 8100 4400
 Wire Wire Line
 	8100 4350 8200 4350
@@
 	4050 5150 5850 5150
 Wire Wire Line
-	2750 4750 2750 4850
+	2750 4750 2750 4800
+Wire Wire Line
+	2750 4800 2750 4850
 Text GLabel 2900 4800 2    60   Input ~ 0
 GND
@@
 GND
 Wire Wire Line
-	5950 7050 6200 7050
+	5950 7050 6050 7050
+Wire Wire Line
+	6050 7050 6200 7050
 Wire Wire Line
 	6200 7250 6050 7250
@@
 	8850 1700 8950 1700
 Text GLabel 5050 5400 2    60   Input ~ 0
-SCLK_5V
+SCLK
 Text GLabel 5050 5500 2    60   Input ~ 0
-MISO_5V
+MISO
 Text GLabel 5050 5600 2    60   Input ~ 0
-MOSI_5V
+MOSI
 Text GLabel 5050 5700 2    60   Input ~ 0
-TFT_CS_5V
+TFT_CS
 Text GLabel 5050 5800 2    60   Input ~ 0
-TFT_DC_5V
+TFT_DC
 Text GLabel 5050 5900 2    60   Input ~ 0
-TOUCH_CS_5V
+TOUCH_CS
 Text GLabel 5050 6200 2    60   Input ~ 0
-SD_CS_5V
+SD_CS
 Wire Wire Line
 	5050 5400 4950 5400
@@
 Wire Wire Line
 	5050 6200 4950 6200
-Text GLabel 3200 6550 2    60   Input ~ 0
-TFT_CS_5V
-Text GLabel 3200 6750 2    60   Input ~ 0
-TOUCH_CS_5V
-Text GLabel 3200 6850 2    60   Input ~ 0
-SD_CS_5V
-Wire Wire Line
-	2950 6550 3200 6550
-Wire Wire Line
-	2950 6650 3200 6650
-Wire Wire Line
-	2950 6750 3200 6750
-Text GLabel 3200 6650 2    60   Input ~ 0
-TFT_DC_5V
-Wire Wire Line
-	3200 6850 2950 6850
 Text GLabel 3200 7150 2    60   Input ~ 0
 SDA_5V
@@
 Wire Wire Line
 	3200 7250 2950 7250
-Text GLabel 3150 6100 2    60   Input ~ 0
-SCLK_5V
-Text GLabel 3150 6200 2    60   Input ~ 0
-MISO_5V
-Text GLabel 3150 6300 2    60   Input ~ 0
-MOSI_5V
-Wire Wire Line
-	3150 6100 2950 6100
-Wire Wire Line
-	3150 6200 2950 6200
-Wire Wire Line
-	3150 6300 2950 6300
-Text GLabel 1300 7150 0    60   Input ~ 0
+Text GLabel 850  7150 0    60   Input ~ 0
 SDA
 Text GLabel 1300 7250 0    60   Input ~ 0
@@
 	1550 7250 1300 7250
 Wire Wire Line
-	1300 7150 1550 7150
-Text GLabel 1300 6100 0    60   Input ~ 0
-SCLK
-Text GLabel 1300 6200 0    60   Input ~ 0
-MISO
-Text GLabel 1300 6300 0    60   Input ~ 0
-MOSI
-Text GLabel 1300 6550 0    60   Input ~ 0
-TFT_CS
-Text GLabel 1300 6650 0    60   Input ~ 0
-TFT_DC
-Text GLabel 1300 6750 0    60   Input ~ 0
-TOUCH_CS
-Text GLabel 1300 6850 0    60   Input ~ 0
-SD_CS
-Wire Wire Line
-	1550 6100 1300 6100
-Wire Wire Line
-	1300 6200 1550 6200
-Wire Wire Line
-	1300 6300 1550 6300
-Wire Wire Line
-	1300 6550 1550 6550
-Wire Wire Line
-	1300 6650 1550 6650
-Wire Wire Line
-	1300 6750 1550 6750
-Wire Wire Line
-	1300 6850 1550 6850
+	850  7150 900  7150
+Wire Wire Line
+	900  7150 1550 7150
 Wire Notes Line
 	550  5100 550  4350
@@
 Wire Notes Line
 	550  5100 650  5100
+Text GLabel 900  7300 3    60   Input ~ 0
+VCC_33
+Wire Wire Line
+	900  7300 900  7150
+Connection ~ 900  7150
 $EndSCHEMATC

Commit message: Updated schematic (solved issues and added Servo)
Parts:
- added P?: CONN_01X03, symbol CONN_01X03
- added R? (x2): 82k, symbol R
Connections:
- net labels added: SERVO_IN, SERVO_OUT
- net labels removed: GPIO_1_D9, VCC33
- wire segments 73 -> 84
Other:
- note added: "Servo BMS 630MG"
Changed lines of the file:
@@
 Text GLabel 5800 1150 2    60   BiDi ~ 0
 LED_VR_IN
-Text GLabel 5800 1250 2    60   BiDi ~ 0
-GPIO_1_D9
 Text GLabel 5800 1350 2    60   BiDi ~ 0
 GND
@@
 $EndComp
 $Sheet
-S 8950 1100 1300 1100
+S 9000 1100 1300 1100
 U 582051C8
 F0 "Ultraschall" 60
 F1 "Ultraschall.sch" 60
-F2 "VCC" I L 8950 1550 60
-F3 "GND" I L 8950 1700 60
-F4 "SDA" B R 10250 1550 60
-F5 "SCL" I R 10250 1700 60
+F2 "VCC" I L 9000 1550 60
+F3 "GND" I L 9000 1700 60
+F4 "SDA" B R 10300 1550 60
+F5 "SCL" I R 10300 1700 60
 $EndSheet
 $Sheet
@@
 GND
 Text GLabel 2900 4650 2    60   Input ~ 0
-VCC33
+VCC_5
 Wire Wire Line
 	2900 4650 2750 4650
@@
 Wire Notes Line
 	550  7750 2500 7750
-Text GLabel 3250 7500 2    60   Input ~ 0
+Text GLabel 3150 7500 2    60   Input ~ 0
 GND
 Text GLabel 1350 5500 0    60   Input ~ 0
-VCC_33
+VCC3P3
 Wire Wire Line
 	1350 5500 1550 5500
 Wire Wire Line
-	3250 7500 2950 7500
+	3150 7500 2950 7500
 Text GLabel 3150 5500 2    60   Input ~ 0
 VCC_5
 Wire Wire Line
 	3150 5500 2950 5500
-Text GLabel 1300 6450 0    60   Input ~ 0
-VCC_33
-Wire Wire Line
-	1300 6450 1550 6450
-Text GLabel 3200 6450 2    60   Input ~ 0
+Text GLabel 1350 6450 0    60   Input ~ 0
+VCC3P3
+Wire Wire Line
+	1350 6450 1550 6450
+Text GLabel 3150 6450 2    60   Input ~ 0
 VCC_5
 Wire Wire Line
-	3200 6450 2950 6450
+	3150 6450 2950 6450
 Wire Notes Line
 	550  5150 4000 5150
@@
 SCL_5V
 Wire Wire Line
-	10400 1550 10250 1550
-Wire Wire Line
-	10400 1700 10250 1700
+	10400 1550 10300 1550
+Wire Wire Line
+	10400 1700 10300 1700
 Text GLabel 8850 1550 0    60   Input ~ 0
 VCC_5
@@
 GND
 Wire Wire Line
-	8850 1550 8950 1550
-Wire Wire Line
-	8850 1700 8950 1700
+	8850 1550 9000 1550
+Wire Wire Line
+	8850 1700 9000 1700
 Text GLabel 5050 5400 2    60   Input ~ 0
 SCLK
@@
 Wire Wire Line
 	5050 6200 4950 6200
-Text GLabel 3200 7150 2    60   Input ~ 0
+Text GLabel 3150 7150 2    60   Input ~ 0
 SDA_5V
-Text GLabel 3200 7250 2    60   Input ~ 0
+Text GLabel 3150 7250 2    60   Input ~ 0
 SCL_5V
 Wire Wire Line
-	3200 7150 2950 7150
-Wire Wire Line
-	3200 7250 2950 7250
+	3150 7150 2950 7150
+Wire Wire Line
+	3150 7250 2950 7250
 Text GLabel 850  7150 0    60   Input ~ 0
 SDA
-Text GLabel 1300 7250 0    60   Input ~ 0
+Text GLabel 850  7250 0    60   Input ~ 0
 SCL
 Wire Wire Line
-	1550 7250 1300 7250
-Wire Wire Line
-	850  7150 900  7150
-Wire Wire Line
-	900  7150 1550 7150
+	850  7250 1250 7250
+Wire Wire Line
+	1250 7250 1550 7250
+Wire Wire Line
+	850  7150 1050 7150
+Wire Wire Line
+	1050 7150 1550 7150
 Wire Notes Line
 	550  5100 550  4350
@@
 Text Notes 600  4450 0    60   ~ 0
 Spannungsversorgung FPGA
-Text GLabel 3200 6950 2    60   Input ~ 0
+Text GLabel 3150 6950 2    60   Input ~ 0
 MOTOR_PWM_5V
 Text GLabel 1350 6950 0    60   Input ~ 0
 MOTOR_PWM_33
-Text GLabel 3200 7050 2    60   Input ~ 0
+Text GLabel 3150 7050 2    60   Input ~ 0
 MOTOR_DIR_5V
 Text GLabel 1350 7050 0    60   Input ~ 0
 MOTOR_DIR_33
 Wire Wire Line
-	3200 6950 2950 6950
-Wire Wire Line
-	3200 7050 2950 7050
+	3150 6950 2950 6950
+Wire Wire Line
+	3150 7050 2950 7050
 Wire Wire Line
 	1550 6950 1350 6950
@@
 Wire Notes Line
 	550  5100 650  5100
-Text GLabel 900  7300 3    60   Input ~ 0
-VCC_33
-Wire Wire Line
-	900  7300 900  7150
-Connection ~ 900  7150
+Text GLabel 950  7650 0    60   Input ~ 0
+VCC3P3
+$Comp
+L R R?
+U 1 1 5828C7A0
+P 1050 7450
+F 0 "R?" V 1130 7450 50  0000 C CNN
+F 1 "82k" V 1050 7450 50  0000 C CNN
+F 2 "" V 980 7450 50  0000 C CNN
+F 3 "" H 1050 7450 50  0000 C CNN
+	1    1050 7450
+	1    0    0    -1
+$EndComp
+$Comp
+L R R?
+U 1 1 5828CA79
+P 1250 7450
+F 0 "R?" V 1330 7450 50  0000 C CNN
+F 1 "82k" V 1250 7450 50  0000 C CNN
+F 2 "" V 1180 7450 50  0000 C CNN
+F 3 "" H 1250 7450 50  0000 C CNN
+	1    1250 7450
+	1    0    0    -1
+$EndComp
+Wire Wire Line
+	1050 7300 1050 7150
+Connection ~ 1050 7150
+Wire Wire Line
+	1250 7300 1250 7250
+Connection ~ 1250 7250
+Wire Wire Line
+	1250 7650 1250 7600
+Wire Wire Line
+	950  7650 1050 7650
+Wire Wire Line
+	1050 7650 1250 7650
+Wire Wire Line
+	1050 7600 1050 7650
+Connection ~ 1050 7650
+Wire Notes Line
+	7250 3800 7250 5100
+Text Notes 6400 3900 0    60   ~ 0
+Servo BMS 630MG
+$Comp
+L CONN_01X03 P?
+U 1 1 582956EF
+P 6800 4950
+F 0 "P?" H 6800 5150 50  0000 C CNN
+F 1 "CONN_01X03" V 6900 4950 50  0000 C CNN
+F 2 "" H 6800 4950 50  0000 C CNN
+F 3 "" H 6800 4950 50  0000 C CNN
+	1    6800 4950
+	0    1    1    0
+$EndComp
+Text GLabel 6900 4500 1    60   Input ~ 0
+GND
+Text GLabel 6800 4500 1    60   Input ~ 0
+VCC_5
+Text GLabel 6700 4500 1    60   Input ~ 0
+SERVO_OUT
+Wire Wire Line
+	6900 4750 6900 4500
+Wire Wire Line
+	6800 4750 6800 4500
+Wire Wire Line
+	6700 4750 6700 4500
+Text GLabel 3150 6300 2    60   Input ~ 0
+SERVO_OUT
+Text GLabel 1350 6300 0    60   Input ~ 0
+SERVO_IN
+Wire Wire Line
+	1350 6300 1550 6300
+Wire Wire Line
+	2950 6300 3150 6300
+Text GLabel 5800 1250 2    60   BiDi ~ 0
+SERVO_IN
+Wire Notes Line
+	7250 5100 6650 5100
+Wire Notes Line
+	6350 5100 6350 3800
+Wire Notes Line
+	6350 3800 7250 3800
+Wire Notes Line
+	6700 5100 6350 5100
 $EndSCHEMATC

Commit message: Updated Schematic
Connections:
- net labels added: LOGIC_OUT, MPU6050_AD0_33, MPU6050_INT_33, MPU6050_XCL_33, MPU6050_XDA_33, ROT_IN, SCL_33, SDA_33
- net labels removed: GPIO_1_D11, GPIO_1_D8
- wire segments 84 -> 97
Other:
- moved on the sheet: P?, R?
