File: Documentation/Schematic/ALF.sch (KiCad schematic (older format))
At the start: 17 parts

Commit message: Updated Schematic (Added USB Port for Router)
Parts:
- added P?: USB_A, symbol USB_A
Other:
- note added: "Spannungsversorgung Router"
- moved on the sheet: R?
Changed lines of the file:
@@
 Text Notes 5950 5250 0    60   ~ 0
 MPU 6050
-Text Notes 4150 6600 0    60   ~ 0
+Text Notes 5650 6600 0    60   ~ 0
 Drehzahlsensor
 Wire Notes Line
@@
 VCC_5
 Wire Wire Line
-	8100 4300 8100 4350
-Wire Wire Line
-	8100 4350 8100 4400
+	8100 4300 8100 4400
 Wire Wire Line
 	8100 4350 8200 4350
@@
 	4050 5150 5850 5150
 Wire Wire Line
-	5150 4800 5150 4850
-Wire Wire Line
-	5150 4850 5150 4900
+	5150 4800 5150 4900
 Text GLabel 5300 4850 2    60   Input ~ 0
 GND
@@
 L CONN_01X04 P?
 U 1 1 58230541
-P 6400 7200
-F 0 "P?" H 6400 7450 50  0000 C CNN
-F 1 "CONN_01X04" V 6500 7200 50  0000 C CNN
-F 2 "" H 6400 7200 50  0000 C CNN
-F 3 "" H 6400 7200 50  0000 C CNN
-	1    6400 7200
+P 6700 7200
+F 0 "P?" H 6700 7450 50  0000 C CNN
+F 1 "CONN_01X04" V 6800 7200 50  0000 C CNN
+F 2 "" H 6700 7200 50  0000 C CNN
+F 3 "" H 6700 7200 50  0000 C CNN
+	1    6700 7200
 	1    0    0    -1
 $EndComp
-Text GLabel 5950 7050 0    60   Input ~ 0
-GND
-Wire Wire Line
-	5950 7050 6050 7050
-Wire Wire Line
-	6050 7050 6200 7050
-Wire Wire Line
-	6200 7250 6050 7250
-Wire Wire Line
-	6050 7250 6050 7050
-Connection ~ 6050 7050
-Text GLabel 5950 7150 0    60   Input ~ 0
+Text GLabel 6100 7050 0    60   Input ~ 0
+GND
+Wire Wire Line
+	6100 7050 6500 7050
+Wire Wire Line
+	6500 7250 6400 7250
+Text GLabel 6100 7150 0    60   Input ~ 0
 VCC_33
-Text GLabel 5250 7350 0    60   Output ~ 0
+Text GLabel 6100 7350 0    60   Output ~ 0
 ROT_OUT
 Wire Wire Line
-	5750 7350 6200 7350
-Wire Wire Line
-	6200 7150 5950 7150
+	6450 7350 6500 7350
+Wire Wire Line
+	6500 7150 6100 7150
 $Comp
 L R R?
 U 1 1 58231B4F
-P 5600 7350
-F 0 "R?" V 5680 7350 50  0000 C CNN
-F 1 "120" V 5600 7350 50  0000 C CNN
-F 2 "" V 5530 7350 50  0000 C CNN
-F 3 "" H 5600 7350 50  0000 C CNN
-	1    5600 7350
+P 6300 7350
+F 0 "R?" V 6380 7350 50  0000 C CNN
+F 1 "120" V 6300 7350 50  0000 C CNN
+F 2 "" V 6230 7350 50  0000 C CNN
+F 3 "" H 6300 7350 50  0000 C CNN
+	1    6300 7350
 	0    1    1    0
 $EndComp
 Wire Wire Line
-	5450 7350 5250 7350
+	6150 7350 6100 7350
 $Sheet
 S 8300 5400 1600 800
@@
 	4000 7750 2450 7750
 Wire Notes Line
-	4050 7750 4050 6500
+	5600 7750 5600 6500
 Wire Notes Line
 	6900 7750 6900 6500
@@
 Wire Notes Line
 	7250 6450 5900 6450
-Wire Notes Line
-	6900 6500 4050 6500
-Wire Notes Line
-	6900 7750 4050 7750
 Text GLabel 4850 550  0    60   Input ~ 0
 VCC3P3
@@
 	5300 950  4850 950
 Wire Wire Line
-	4850 550  5000 550
-Wire Wire Line
-	5000 550  5200 550
+	4850 550  5200 550
 Wire Wire Line
 	5200 550  5200 650
@@
 Wire Wire Line
 	3100 7150 2900 7150
+Wire Wire Line
+	6400 7250 6400 7050
+Connection ~ 6400 7050
+Wire Notes Line
+	6900 6500 5600 6500
+Wire Notes Line
+	5600 7750 6900 7750
+Wire Notes Line
+	4050 6500 5550 6500
+Wire Notes Line
+	5550 6500 5550 7750
+Wire Notes Line
+	5550 7750 4050 7750
+Wire Notes Line
+	4050 7750 4050 6500
+Text Notes 4100 6600 0    60   ~ 0
+Spannungsversorgung Router
+$Comp
+L USB_A P?
+U 1 1 58338FBE
+P 4800 6900
+F 0 "P?" H 5000 6700 50  0000 C CNN
+F 1 "USB_A" H 4750 7100 50  0000 C CNN
+F 2 "" V 4750 6800 50  0000 C CNN
+F 3 "" V 4750 6800 50  0000 C CNN
+	1    4800 6900
+	1    0    0    -1
+$EndComp
+Text GLabel 4900 7300 3    60   Input ~ 0
+GND
+Text GLabel 4600 7300 3    60   Input ~ 0
+VCC_5
+Wire Wire Line
+	4900 7300 4900 7200
+Wire Wire Line
+	4600 7200 4600 7300
+Wire Wire Line
+	5100 6800 5100 7250
+Wire Wire Line
+	5100 7250 4900 7250
+Connection ~ 4900 7250
 $EndSCHEMATC

Commit message: Annotated Schematic
Parts:
- gave numbers to parts that had none: 11
Changed lines of the file:
@@
 LIBS:contrib
 LIBS:valves
-LIBS:ALF-cache
 EELAYER 25 0
 EELAYER END
@@
 $EndComp
 $Comp
-L CONN_02X05 P?
+L CONN_02X05 P1
 U 1 1 58171862
 P 1400 3550
-F 0 "P?" H 1400 3850 50  0000 C CNN
+F 0 "P1" H 1400 3850 50  0000 C CNN
 F 1 "CONN_02X05" H 1400 3250 50  0000 C CNN
 F 2 "" H 1400 2350 50  0000 C CNN
@@
 $EndComp
 $Comp
-L CONN_02X07 P?
+L CONN_02X07 P3
 U 1 1 581718D6
 P 5550 3300
-F 0 "P?" H 5550 3700 50  0000 C CNN
+F 0 "P3" H 5550 3700 50  0000 C CNN
 F 1 "CONN_02X07" V 5550 3300 50  0000 C CNN
 F 2 "" H 5550 2100 50  0000 C CNN
@@
 GND
 $Comp
-L GND #PWR?
+L GND #PWR1
 U 1 1 5818C15E
 P 7750 1100
-F 0 "#PWR?" H 7750 850 50  0001 C CNN
+F 0 "#PWR1" H 7750 850 50  0001 C CNN
 F 1 "GND" H 7750 950 50  0000 C CNN
 F 2 "" H 7750 1100 50  0000 C CNN
@@
 Spannungswandler
 $Comp
-L BARREL_JACK CON?
+L BARREL_JACK CON1
 U 1 1 58205FBE
 P 4850 4800
-F 0 "CON?" H 4850 5050 50  0000 C CNN
+F 0 "CON1" H 4850 5050 50  0000 C CNN
 F 1 "BARREL_JACK" H 4850 4600 50  0000 C CNN
 F 2 "" H 4850 4800 50  0000 C CNN
@@
 $EndSheet
 $Comp
-L CONN_01X02 P?
+L CONN_01X02 P7
 U 1 1 582235DE
 P 7900 4450
-F 0 "P?" H 7900 4600 50  0000 C CNN
+F 0 "P7" H 7900 4600 50  0000 C CNN
 F 1 "CONN_AKKU" V 8000 4450 50  0000 C CNN
 F 2 "" H 7900 4450 50  0000 C CNN
@@
 Connection ~ 5150 4850
 $Comp
-L CONN_01X08 P?
+L CONN_01X08 P6
 U 1 1 5822E87F
 P 7100 5800
-F 0 "P?" H 7100 6250 50  0000 C CNN
+F 0 "P6" H 7100 6250 50  0000 C CNN
 F 1 "CONN_01X08" V 7200 5800 50  0000 C CNN
 F 2 "" H 7100 5800 50  0000 C CNN
@@
 	6750 6150 6900 6150
 $Comp
-L CONN_01X04 P?
+L CONN_01X04 P4
 U 1 1 58230541
 P 6700 7200
-F 0 "P?" H 6700 7450 50  0000 C CNN
+F 0 "P4" H 6700 7450 50  0000 C CNN
 F 1 "CONN_01X04" V 6800 7200 50  0000 C CNN
 F 2 "" H 6700 7200 50  0000 C CNN
@@
 	6500 7150 6100 7150
 $Comp
-L R R?
+L R R3
 U 1 1 58231B4F
 P 6300 7350
-F 0 "R?" V 6380 7350 50  0000 C CNN
+F 0 "R3" V 6380 7350 50  0000 C CNN
 F 1 "120" V 6300 7350 50  0000 C CNN
 F 2 "" V 6230 7350 50  0000 C CNN
@@
 VCC3P3
 $Comp
-L R R?
+L R R2
 U 1 1 5828C7A0
 P 5200 800
-F 0 "R?" V 5280 800 50  0000 C CNN
+F 0 "R2" V 5280 800 50  0000 C CNN
 F 1 "82k" V 5200 800 50  0000 C CNN
 F 2 "" V 5130 800 50  0000 C CNN
@@
 $EndComp
 $Comp
-L R R?
+L R R1
 U 1 1 5828CA79
 P 5000 700
-F 0 "R?" V 5080 700 50  0000 C CNN
+F 0 "R1" V 5080 700 50  0000 C CNN
 F 1 "82k" V 5000 700 50  0000 C CNN
 F 2 "" V 4930 700 50  0000 C CNN
@@
 Servo BMS 630MG
 $Comp
-L CONN_01X03 P?
+L CONN_01X03 P5
 U 1 1 582956EF
 P 6800 4950
-F 0 "P?" H 6800 5150 50  0000 C CNN
+F 0 "P5" H 6800 5150 50  0000 C CNN
 F 1 "CONN_01X03" V 6900 4950 50  0000 C CNN
 F 2 "" H 6800 4950 50  0000 C CNN
@@
 Spannungsversorgung Router
 $Comp
-L USB_A P?
+L USB_A P2
 U 1 1 58338FBE
 P 4800 6900
-F 0 "P?" H 5000 6700 50  0000 C CNN
+F 0 "P2" H 5000 6700 50  0000 C CNN
 F 1 "USB_A" H 4750 7100 50  0000 C CNN
 F 2 "" V 4750 6800 50  0000 C CNN

Commit message: Changed Label SERVO_IN and SERVO_OUT to STEERING_CONTROL_IN and STEERING_CONTROL_OUT
Connections:
- net labels added: STEERING_CONTROL_IN, STEERING_CONTROL_OUT
- net labels removed: SERVO_IN, SERVO_OUT
Other:
- note added: "Spannungsversorgung\nFPGA"
- note removed: "Spannungsversorgung FPGA"
- moved on the sheet: P6, R3
