File: Documentation/Schematic/Beleuchtung.sch (KiCad schematic (older format))
At the start: 8 parts

Commit message: Annotated Schematic
Parts:
- gave numbers to parts that had none: 8
Changed lines of the file:
@@
 LIBS:contrib
 LIBS:valves
-LIBS:ALF-cache
 EELAYER 25 0
 EELAYER END
@@
 GND
 $Comp
-L LED D?
+L LED D1
 U 1 1 582079CB
 P 2550 3050
-F 0 "D?" H 2550 3150 50  0000 C CNN
+F 0 "D1" H 2550 3150 50  0000 C CNN
 F 1 "LED" H 2550 2950 50  0000 C CNN
 F 2 "" H 2550 3050 50  0000 C CNN
@@
 $EndComp
 $Comp
-L R R?
+L R R4
 U 1 1 582079F7
 P 2550 2700
-F 0 "R?" V 2630 2700 50  0000 C CNN
+F 0 "R4" V 2630 2700 50  0000 C CNN
 F 1 "R" V 2550 2700 50  0000 C CNN
 F 2 "" V 2480 2700 50  0000 C CNN
@@
 GND
 $Comp
-L LED D?
+L LED D2
 U 1 1 58207A7E
 P 3150 3050
-F 0 "D?" H 3150 3150 50  0000 C CNN
+F 0 "D2" H 3150 3150 50  0000 C CNN
 F 1 "LED" H 3150 2950 50  0000 C CNN
 F 2 "" H 3150 3050 50  0000 C CNN
@@
 $EndComp
 $Comp
-L R R?
+L R R5
 U 1 1 58207A84
 P 3150 2700
-F 0 "R?" V 3230 2700 50  0000 C CNN
+F 0 "R5" V 3230 2700 50  0000 C CNN
 F 1 "R" V 3150 2700 50  0000 C CNN
 F 2 "" V 3080 2700 50  0000 C CNN
@@
 GND
 $Comp
-L LED D?
+L LED D3
 U 1 1 58207AFC
 P 3750 3050
-F 0 "D?" H 3750 3150 50  0000 C CNN
+F 0 "D3" H 3750 3150 50  0000 C CNN
 F 1 "LED" H 3750 2950 50  0000 C CNN
 F 2 "" H 3750 3050 50  0000 C CNN
@@
 $EndComp
 $Comp
-L R R?
+L R R6
 U 1 1 58207B02
 P 3750 2700
-F 0 "R?" V 3830 2700 50  0000 C CNN
+F 0 "R6" V 3830 2700 50  0000 C CNN
 F 1 "R" V 3750 2700 50  0000 C CNN
 F 2 "" V 3680 2700 50  0000 C CNN
@@
 GND
 $Comp
-L LED D?
+L LED D4
 U 1 1 58207B74
 P 4300 3050
-F 0 "D?" H 4300 3150 50  0000 C CNN
+F 0 "D4" H 4300 3150 50  0000 C CNN
 F 1 "LED" H 4300 2950 50  0000 C CNN
 F 2 "" H 4300 3050 50  0000 C CNN
@@
 $EndComp
 $Comp
-L R R?
+L R R7
 U 1 1 58207B7A
 P 4300 2700
-F 0 "R?" V 4380 2700 50  0000 C CNN
+F 0 "R7" V 4380 2700 50  0000 C CNN
 F 1 "R" V 4300 2700 50  0000 C CNN
 F 2 "" V 4230 2700 50  0000 C CNN

Commit message: Updated Schematic to match with Lighting circuit (Removed not used IIC pull-ups also)
Parts:
- D1, D2, D3, D4: symbol LED -> LED-RESCUE-ALF
- R4, R5, R6, R7: symbol R -> R-RESCUE-ALF
Connections:
- net LED_HR is gone; now on net 5V: R6.1
- net LED_VL is gone; now on net 5V: R5.1
- net LED_VR is gone; now on net 5V: R4.1
- net at D1.2 (K): no longer R4.2
- net at D2.2 (K): no longer R5.2
- net at D3.2 (K): no longer R6.2
- net at D4.2 (K): no longer R7.2
- net GND renamed LED
- net LED_HL renamed 5V
Other:
- note added: "Low active circuit"
Changed lines of the file:
@@
 EESchema Schematic File Version 2
+LIBS:ALF-rescue
 LIBS:power
 LIBS:device
@@
 LIBS:contrib
 LIBS:valves
+LIBS:ALF-cache
 EELAYER 25 0
 EELAYER END
@@
 Comment4 ""
 $EndDescr
-Text HLabel 2550 3250 3    60   Input ~ 0
-GND
 $Comp
-L LED D1
+L LED-RESCUE-ALF D1
 U 1 1 582079CB
 P 2550 3050
+AR Path="/582079CB" Ref="D1"  Part="1"
+AR Path="/58207938/582079CB" Ref="D1"  Part="1"
 F 0 "D1" H 2550 3150 50  0000 C CNN
 F 1 "LED" H 2550 2950 50  0000 C CNN
@@
 $EndComp
 $Comp
-L R R4
+L R-RESCUE-ALF R4
 U 1 1 582079F7
 P 2550 2700
+AR Path="/582079F7" Ref="R4"  Part="1"
+AR Path="/58207938/582079F7" Ref="R4"  Part="1"
 F 0 "R4" V 2630 2700 50  0000 C CNN
 F 1 "R" V 2550 2700 50  0000 C CNN
@@
 	1    0    0    -1
 $EndComp
-Text HLabel 2550 2550 1    60   Input ~ 0
-LED_VR
-Text HLabel 3150 3250 3    60   Input ~ 0
-GND
 $Comp
-L LED D2
+L LED-RESCUE-ALF D2
 U 1 1 58207A7E
 P 3150 3050
+AR Path="/58207A7E" Ref="D2"  Part="1"
+AR Path="/58207938/58207A7E" Ref="D2"  Part="1"
 F 0 "D2" H 3150 3150 50  0000 C CNN
 F 1 "LED" H 3150 2950 50  0000 C CNN
@@
 $EndComp
 $Comp
-L R R5
+L R-RESCUE-ALF R5
 U 1 1 58207A84
 P 3150 2700
+AR Path="/58207A84" Ref="R5"  Part="1"
+AR Path="/58207938/58207A84" Ref="R5"  Part="1"
 F 0 "R5" V 3230 2700 50  0000 C CNN
 F 1 "R" V 3150 2700 50  0000 C CNN
@@
 	1    0    0    -1
 $EndComp
-Text HLabel 3150 2550 1    60   Input ~ 0
-LED_VL
-Text HLabel 3750 3250 3    60   Input ~ 0
-GND
 $Comp
-L LED D3
+L LED-RESCUE-ALF D3
 U 1 1 58207AFC
 P 3750 3050
+AR Path="/58207AFC" Ref="D3"  Part="1"
+AR Path="/58207938/58207AFC" Ref="D3"  Part="1"
 F 0 "D3" H 3750 3150 50  0000 C CNN
 F 1 "LED" H 3750 2950 50  0000 C CNN
@@
 $EndComp
 $Comp
-L R R6
+L R-RESCUE-ALF R6
 U 1 1 58207B02
 P 3750 2700
+AR Path="/58207B02" Ref="R6"  Part="1"
+AR Path="/58207938/58207B02" Ref="R6"  Part="1"
 F 0 "R6" V 3830 2700 50  0000 C CNN
 F 1 "R" V 3750 2700 50  0000 C CNN
@@
 	1    0    0    -1
 $EndComp
-Text HLabel 3750 2550 1    60   Input ~ 0
-LED_HR
-Text HLabel 4300 3250 3    60   Input ~ 0
-GND
 $Comp
-L LED D4
+L LED-RESCUE-ALF D4
 U 1 1 58207B74
 P 4300 3050
+AR Path="/58207B74" Ref="D4"  Part="1"
+AR Path="/58207938/58207B74" Ref="D4"  Part="1"
 F 0 "D4" H 4300 3150 50  0000 C CNN
 F 1 "LED" H 4300 2950 50  0000 C CNN
@@
 $EndComp
 $Comp
-L R R7
+L R-RESCUE-ALF R7
 U 1 1 58207B7A
 P 4300 2700
+AR Path="/58207B7A" Ref="R7"  Part="1"
+AR Path="/58207938/58207B7A" Ref="R7"  Part="1"
 F 0 "R7" V 4380 2700 50  0000 C CNN
 F 1 "R" V 4300 2700 50  0000 C CNN
@@
 	1    0    0    -1
 $EndComp
-Text HLabel 4300 2550 1    60   Input ~ 0
-LED_HL
+Wire Wire Line
+	2550 3250 4300 3250
+Connection ~ 3150 3250
+Connection ~ 3750 3250
+Wire Wire Line
+	3450 3250 3450 3350
+Connection ~ 3450 3250
+Text HLabel 3450 3350 3    60   Input ~ 0
+LED
+Wire Wire Line
+	2550 2450 4300 2450
+Connection ~ 3150 2450
+Connection ~ 3750 2450
+Wire Wire Line
+	3450 2450 3450 2350
+Connection ~ 3450 2450
+Text HLabel 3450 2350 1    60   Input ~ 0
+5V
+Text Notes 3350 2100 2    60   ~ 0
+Low active circuit
 $EndSCHEMATC
