File: Documentation/Schematic/Display.sch (KiCad schematic (older format))
At the start: 4 parts

Commit message: Annotated Schematic
Parts:
- gave numbers to parts that had none: 4
Changed lines of the file:
@@
 LIBS:contrib
 LIBS:valves
-LIBS:ALF-cache
 EELAYER 25 0
 EELAYER END
@@
 $EndDescr
 $Comp
-L CONN_01X08 P?
+L CONN_01X08 P14
 U 1 1 5827A7DB
 P 2600 1550
-F 0 "P?" H 2600 2000 50  0000 C CNN
+F 0 "P14" H 2600 2000 50  0000 C CNN
 F 1 "CONN_01X08" V 2700 1550 50  0000 C CNN
 F 2 "" H 2600 1550 50  0000 C CNN
@@
 $EndComp
 $Comp
-L CONN_01X06 P?
+L CONN_01X06 P15
 U 1 1 5827A80C
 P 2600 2350
-F 0 "P?" H 2600 2700 50  0000 C CNN
+F 0 "P15" H 2600 2700 50  0000 C CNN
 F 1 "CONN_01X06" V 2700 2350 50  0000 C CNN
 F 2 "" H 2600 2350 50  0000 C CNN
@@
 $EndComp
 $Comp
-L CONN_01X10 P?
+L CONN_01X10 P16
 U 1 1 5827A835
 P 4100 1350
-F 0 "P?" H 4100 1900 50  0000 C CNN
+F 0 "P16" H 4100 1900 50  0000 C CNN
 F 1 "CONN_01X10" V 4200 1350 50  0000 C CNN
 F 2 "" H 4100 1350 50  0000 C CNN
@@
 $EndComp
 $Comp
-L CONN_01X08 P?
+L CONN_01X08 P17
 U 1 1 5827A8EE
 P 4100 2350
-F 0 "P?" H 4100 2800 50  0000 C CNN
+F 0 "P17" H 4100 2800 50  0000 C CNN
 F 1 "CONN_01X08" V 4200 2350 50  0000 C CNN
 F 2 "" H 4100 2350 50  0000 C CNN
