File: Documentation/Schematic/Levelshifter.sch (KiCad schematic (older format))
At the start: 2 parts

Commit message: Updated hierarchical sheet Levelshifter
Parts:
- added P?: Levelshifter3, symbol CONN_02X10
Connections:
- net labels added: A31, A32, A33, A34, A35, A36, A37, A38, B31, B32, B33, B34, B35, B36, B37, B38, OE3, VCC3A, VCC3B
Changed lines of the file:
@@
 LIBS:contrib
 LIBS:valves
-LIBS:ALF-cache
 EELAYER 25 0
 EELAYER END
 $Descr A4 11693 8268
 encoding utf-8
-Sheet 6 7
+Sheet 7 7
 Title ""
 Date ""
@@
 Text HLabel 3450 2150 2    60   Input ~ 0
 GND
+$Comp
+L CONN_02X10 P?
+U 1 1 5829D056
+P 4600 1700
+F 0 "P?" H 4600 2250 50  0000 C CNN
+F 1 "Levelshifter3" V 4600 1700 50  0000 C CNN
+F 2 "" H 4600 500 50  0000 C CNN
+F 3 "" H 4600 500 50  0000 C CNN
+	1    4600 1700
+	1    0    0    -1
+$EndComp
+Text HLabel 4350 1350 0    60   Input ~ 0
+VCC3A
+Text HLabel 4350 1250 0    60   BiDi ~ 0
+A31
+Text HLabel 4350 1450 0    60   BiDi ~ 0
+A32
+Text HLabel 4350 1550 0    60   BiDi ~ 0
+A33
+Text HLabel 4350 1650 0    60   BiDi ~ 0
+A34
+Text HLabel 4350 1750 0    60   BiDi ~ 0
+A35
+Text HLabel 4350 1850 0    60   BiDi ~ 0
+A36
+Text HLabel 4350 1950 0    60   BiDi ~ 0
+A37
+Text HLabel 4350 2050 0    60   BiDi ~ 0
+A38
+Text HLabel 4350 2150 0    60   Input ~ 0
+OE3
+Text HLabel 4850 1250 2    60   BiDi ~ 0
+B31
+Text HLabel 4850 1350 2    60   Input ~ 0
+VCC3B
+Text HLabel 4850 1450 2    60   BiDi ~ 0
+B32
+Text HLabel 4850 1550 2    60   BiDi ~ 0
+B33
+Text HLabel 4850 1650 2    60   BiDi ~ 0
+B34
+Text HLabel 4850 1750 2    60   BiDi ~ 0
+B35
+Text HLabel 4850 1850 2    60   BiDi ~ 0
+B36
+Text HLabel 4850 1950 2    60   BiDi ~ 0
+B37
+Text HLabel 4850 2050 2    60   BiDi ~ 0
+B38
+Text HLabel 4850 2150 2    60   Input ~ 0
+GND
 $EndSCHEMATC

Commit message: Annotated Schematic
Parts:
- gave numbers to parts that had none: 3
Changed lines of the file:
@@
 LIBS:contrib
 LIBS:valves
-LIBS:ALF-cache
 EELAYER 25 0
 EELAYER END
@@
 $EndDescr
 $Comp
-L CONN_02X10 P?
+L CONN_02X10 P18
 U 1 1 5823B5BC
 P 1850 1700
-F 0 "P?" H 1850 2250 50  0000 C CNN
+F 0 "P18" H 1850 2250 50  0000 C CNN
 F 1 "Levelshifter1" V 1850 1700 50  0000 C CNN
 F 2 "" H 1850 500 50  0000 C CNN
@@
 GND
 $Comp
-L CONN_02X10 P?
+L CONN_02X10 P19
 U 1 1 5823B6A1
 P 3200 1700
-F 0 "P?" H 3200 2250 50  0000 C CNN
+F 0 "P19" H 3200 2250 50  0000 C CNN
 F 1 "Levelshifter2" V 3200 1700 50  0000 C CNN
 F 2 "" H 3200 500 50  0000 C CNN
@@
 GND
 $Comp
-L CONN_02X10 P?
+L CONN_02X10 P20
 U 1 1 5829D056
 P 4600 1700
-F 0 "P?" H 4600 2250 50  0000 C CNN
+F 0 "P20" H 4600 2250 50  0000 C CNN
 F 1 "Levelshifter3" V 4600 1700 50  0000 C CNN
 F 2 "" H 4600 500 50  0000 C CNN
