File: Documentation/Schematic/Spannungswandler.sch (KiCad schematic (older format))
At the start: 2 parts

Commit message: Annotated Schematic
Parts:
- gave numbers to parts that had none: 2
Changed lines of the file:
@@
 LIBS:contrib
 LIBS:valves
-LIBS:ALF-cache
 EELAYER 25 0
 EELAYER END
@@
 $EndDescr
 $Comp
-L CONN_01X03 P?
+L CONN_01X03 P12
 U 1 1 5822507B
 P 2000 1200
-F 0 "P?" H 2000 1400 50  0000 C CNN
+F 0 "P12" H 2000 1400 50  0000 C CNN
 F 1 "CONN_01X03" V 2100 1200 50  0000 C CNN
 F 2 "" H 2000 1200 50  0000 C CNN
@@
 $EndComp
 $Comp
-L CONN_01X03 P?
+L CONN_01X03 P13
 U 1 1 582250EA
 P 3050 1200
-F 0 "P?" H 3050 1400 50  0000 C CNN
+F 0 "P13" H 3050 1400 50  0000 C CNN
 F 1 "CONN_01X03" V 3150 1200 50  0000 C CNN
 F 2 "" H 3050 1200 50  0000 C CNN
