File: Documentation/Schematic/Ultraschall.sch (KiCad schematic (older format))
At the start: 4 parts

Commit message: Annotated Schematic
Parts:
- gave numbers to parts that had none: 4
Changed lines of the file:
@@
 LIBS:contrib
 LIBS:valves
-LIBS:ALF-cache
 EELAYER 25 0
 EELAYER END
@@
 $EndDescr
 $Comp
-L CONN_01X05 P?
+L CONN_01X05 P8
 U 1 1 582053A3
 P 2700 1800
-F 0 "P?" H 2700 2100 50  0000 C CNN
+F 0 "P8" H 2700 2100 50  0000 C CNN
 F 1 "CONN_01X05" V 2800 1800 50  0000 C CNN
 F 2 "" H 2700 1800 50  0000 C CNN
@@
 $EndComp
 $Comp
-L CONN_01X05 P?
+L CONN_01X05 P9
 U 1 1 58205436
 P 2700 3350
-F 0 "P?" H 2700 3650 50  0000 C CNN
+F 0 "P9" H 2700 3650 50  0000 C CNN
 F 1 "CONN_01X05" V 2800 3350 50  0000 C CNN
 F 2 "" H 2700 3350 50  0000 C CNN
@@
 $EndComp
 $Comp
-L CONN_01X05 P?
+L CONN_01X05 P10
 U 1 1 5820546D
 P 5550 1800
-F 0 "P?" H 5550 2100 50  0000 C CNN
+F 0 "P10" H 5550 2100 50  0000 C CNN
 F 1 "CONN_01X05" V 5650 1800 50  0000 C CNN
 F 2 "" H 5550 1800 50  0000 C CNN
@@
 $EndComp
 $Comp
-L CONN_01X05 P?
+L CONN_01X05 P11
 U 1 1 5820548E
 P 5550 3300
-F 0 "P?" H 5550 3600 50  0000 C CNN
+F 0 "P11" H 5550 3600 50  0000 C CNN
 F 1 "CONN_01X05" V 5650 3300 50  0000 C CNN
 F 2 "" H 5550 3300 50  0000 C CNN
